File: pico-dram-tester.kicad_pcb (KiCad board)
At the start: 2 copper layers, 100 x 100 mm, 44 parts, among them J1 TFT 4383, J2 mrd_114_ips_lcd_8p, Q1 2N3906, SW1 RotaryEncoder_Switch, SW2 BACK, U1 PICO2, U2 4116, U3 4132, U4 4164/41128/41256, U5 4416/4464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

Commit message: Layout corrections
Parts:
- Q1: value 2N3906 -> XP9561GI; footprint Package_TO_SOT_THT:TO-92_Inline_Wide -> Package_TO_SOT_THT:TO-220-3_Vertical
- R5: value 4.7K -> 100
- moved Q1 4.35 mm to (155.2, 68.7), turned to 90 degrees
Connections:
- Q1 pad 1: VCC -> Net-(Q1-G)
- Q1 pad 2: Net-(Q1-B) -> +5V
- Q1 pad 3: +5V -> VCC
- R4 pad 2: Net-(Q1-B) -> Net-(Q1-G)
- R5 pad 1: Net-(Q1-B) -> Net-(Q1-G)
Routing:
- net Net-(Q1-G): track 0.00 -> 8.34 mm
- net Net-(Q1-B): track 7.64 -> 0.00 mm
- net /SP9: track 172.9 -> 174.8 mm
- net VCC: track 146.6 -> 147.5 mm
- net GND: vias 181 -> 189
Other:
- board text added: "Rev 2 11/24"
- board text removed: "Rev 1 10/24"

Commit message: DCJack and Generic Encoder
Added DC Barrel Jack. Added Configuration Jumper pads to use the common Generic Encoder
Parts:
- removed TP6: GND, TestPoint:TestPoint_Keystone_5005-5009_Compact
- added J3: 5V DC Jack, Connector_BarrelJack:BarrelJack_Horizontal, F.Cu at (143.0, 60.5)
- added JP1: EncoderCFG, Jumper:SolderJumper-3_P1.3mm_Open_Pad1.0x1.5mm, F.Cu at (120.6, 144.8)
- Q1: value XP9561GI -> SUP53P06-20-E3 or equiv
- R1, RN1, RN2, RN3, RN4: value 100 -> 33
- moved C1 11.3 mm to (150.2, 58.5)
- moved TP4 8.85 mm to (150.0, 54.5)
- moved TP1 3.43 mm to (155.6, 54.5)
- moved TP3 3.23 mm to (161.0, 54.5)
- moved TP2 2.03 mm to (134.2, 54.5)
- moved TP5 1.16 mm to (103.6, 54.5)
Connections:
- RN3 pad 3: /SP9 -> +5V
- U2 pad 2: /SP9 -> +5V
- U3 pad 2: /SP9 -> +5V
- U4 pad 2: /SP9 -> +5V
- U5 pad 8: /SP9 -> +5V
- U6 pad 11: /SP9 -> +5V
Routing:
- net /SP9: track 174.8 -> 0.00 mm, vias 2 -> 0
- net +5V: track 176.3 -> 350.7 mm, vias 0 -> 2
- net Net-(JP1-C): track 0.00 -> 10.6 mm
- net VCC: track 147.5 -> 155.0 mm, vias 1 -> 2
- net Net-(JP1-A): track 97.4 -> 104.6 mm
- net -5V: track 106.9 -> 112.8 mm
- net /SP4: track 241.9 -> 245.3 mm
- net +3V3: track 116.2 -> 113.6 mm
- net /SP0: track 196.9 -> 199.1 mm
- net +12V: track 133.4 -> 135.5 mm
- net /SP16: track 128.9 -> 127.5 mm
- net /SP3: track 219.5 -> 220.7 mm
- net /SP12: track 153.8 -> 154.7 mm
- net /SP10: track 169.8 -> 168.9 mm
- net /SP8: track 115.2 -> 116.0 mm
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Other:
- board text added: "JP1 Encoder Config: Pad 1 & 2 = Panasonic EVE-YBCAJO16B Pad 2 & 3 = Generic Encoder"
- board text added: "Rev 2.2 8/25"
- board text removed: "Rev 2 11/24"
